Commit message: Toco volver a plan inicial de controlar el robot con python

File: src/burger1_description/resource/burger1.urdf.xacro (robot description, xacro)
@@ -2,6 +2,4 @@
 <robot xmlns:xacro="http://www.ros.org/wiki/xacro"  name="robot">
     <xacro:include filename="base_link.xacro"/>
-    <!-- Se sustituye por ros2_control -->
-    <!-- <xacro:include filename="gazebo_control.xacro"/> -->
     <xacro:include filename="ros2_control.xacro"/>
 </robot>

File: src/burger1_description/resource/ros2_control.xacro (robot description, xacro)
@@ -1,28 +1,5 @@
 <?xml version="1.0"?>
 <robot xmlns:xacro="http://www.ros.org/wiki/xacro">
-    <ros2_control name="RealRobot" type="system">
-        <hardware>
-            <plugin>burger1_robot/DiffBotSystemHardware</plugin>
-            <param name="example_param_hw_start_duration_sec">0</param>
-            <param name="example_param_hw_stop_duration_sec">3.0</param>
-        </hardware>
-        <joint name="left_wheel_joint">
-            <command_interface name="velocity">
-                <param name="min">-10</param>
-                <param name="max">10</param>
-            </command_interface>
-            <state_interface name="velocity"/>
-            <state_interface name="position"/>
-        </joint>
-        <joint name="right_wheel_joint">
-            <command_interface name="velocity">
-                <param name="min">-10</param>
-                <param name="max">10</param>
-            </command_interface>
-            <state_interface name="velocity"/>
-            <state_interface name="position"/>
-        </joint>
-    </ros2_control>
-    <!-- <ros2_control name="GazeboSystem" type="system">
+    <ros2_control name="GazeboSystem" type="system">
         <hardware>
             <plugin>gazebo_ros2_control/GazeboSystem</plugin>
@@ -44,5 +21,5 @@
             <state_interface name="position"/>
         </joint>
-    </ros2_control> -->
+    </ros2_control>
     <gazebo>
         <plugin name="gazebo_ros2_control" filename="libgazebo_ros2_control.so">
